File: BBB_Pololu.kicad_pcb (KiCad board)
At the start: 2 copper layers, 90 x 45 mm, 26 parts, among them J0 CONN_01X04, J1 CONN_01X04, J2 CONN_01X04, P1 VM_IN, P2 CONN_02X03, P4 CONN_02X03, P6 CONN_02X03, P8 AXIS_LED, P9 LED_VM, Q1 2N7002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

Commit message: Routed but checks to be done
Parts:
- moved R3 68.1 mm to (93.0, 124.0), turned to 270 degrees
- moved R4 57.9 mm to (103.1, 126.1), turned to 90 degrees
- moved Q1 56.5 mm to (97.5, 126.8), turned to 90 degrees
- moved R6 27.4 mm to (83.0, 118.1), turned to 270 degrees
- moved P9 11.9 mm to (83.1, 123.8), turned to 270 degrees
- moved R1 9.93 mm to (97.9, 130.6), turned to 180 degrees
- moved Q2 9.90 mm to (97.6, 122.7), turned to 90 degrees
- moved P8 9.41 mm to (88.6, 124.1)
- moved U1 7.00 mm to (168.0, 128.0)
- moved R5 6.66 mm to (92.1, 130.6), turned to 180 degrees
- moved TPGnd1 3.54 mm to (84.4, 130.4)
- moved R2 1.25 mm to (87.4, 118.1), turned to 270 degrees
- moved J1 0.54 mm to (140.5, 110.2)
Routing:
- net GND: track 0.00 -> 232.3 mm, vias 0 -> 3
- net +3V3: track 0.00 -> 160.0 mm, vias 0 -> 3
- net /Vm: track 0.00 -> 129.8 mm
- net AXIS_ENB: track 0.00 -> 90.2 mm, vias 0 -> 4
- net AXIS_EN: track 0.00 -> 58.7 mm
- net STEP_2: track 0.00 -> 54.9 mm
- net ESTOP: track 0.00 -> 53.7 mm
- net DIR_2: track 0.00 -> 50.7 mm
- net STEP_1: track 0.00 -> 35.6 mm
- net DIR_1: track 0.00 -> 32.8 mm
- net STEP_0: track 0.00 -> 18.7 mm
- net DIR_0: track 0.00 -> 15.0 mm
- net Net-(P8-Pad1): track 0.00 -> 10.5 mm
- net Net-(J2-Pad4): track 0.00 -> 9.82 mm
- net Net-(J1-Pad2): track 0.00 -> 9.78 mm
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- added copper zone on B.Cu, net GND
Other:
- board size 90 x 45 mm -> 90 x 38 mm
- board text added: "ToDo: Silk screen meaningful Axis and motor directions, polarities Check pin sizes and anular rings on pin headers + pololu"

Commit message: Silk not finished
Parts:
- moved R2 1.10 mm to (88.5, 118.0)
- moved P9 0.22 mm to (83.0, 124.0)
- renumbered TPGnd1 to Gnd
Routing:
- net Net-(R2-Pad1): track 4.79 -> 6.07 mm
- net ESTOP: track 53.7 -> 52.6 mm
Other:
- board text added: "+Enb"
- board text added: "EStop"
- board text added: "Mtr +"
- board text added: "Vmtr"
- board text added: "X"
- board text added: "Y"
- board text added: "Z"
- board text removed: "ToDo: Silk screen meaningful Axis and motor directions, polarities Check pin sizes and anular rings on pin headers + pololu"

Commit message: As sent for manufacture
Other:
- board text added: "0"
- board text added: "1"
- board text added: "2"
- board text added: "BBB -> Pololu"
Changed lines of the file:
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@@
-(kicad_pcb (version 4) (host pcbnew 4.0.1-stable)
+(kicad_pcb (version 4) (host pcbnew 4.0.2-stable)
   (general
     (links 85)
     (no_connects 0)
-    (area 55.8 85.4 171.475 134.6192)
+    (area 77.860067 94.924999 171.475 134.6192)
     (thickness 1.6)
-    (drawings 11)
+    (drawings 27)
     (tracks 316)
     (zones 0)
@@
   )
   (setup
-    (last_trace_width 0.4)
+    (last_trace_width 0.25)
     (user_trace_width 0.2)
     (user_trace_width 0.25)
@@
     (visible_elements 7FFEFF7F)
     (pcbplotparams
-      (layerselection 0x00030_80000001)
-      (usegerberextensions false)
+      (layerselection 0x010f0_80000001)
+      (usegerberextensions true)
       (excludeedgelayer true)
       (linewidth 0.100000)
@@
       (psa4output false)
       (plotreference true)
-      (plotvalue true)
+      (plotvalue false)
       (plotinvisibletext false)
       (padsonsilk false)
@@
       (outputformat 1)
       (mirror false)
-      (drillshape 1)
+      (drillshape 0)
       (scaleselection 1)
-      (outputdirectory ""))
+      (outputdirectory Gerb/))
   )
   (net 0 "")
@@
     (descr "1 pin")
     (tags "CONN DEV")
-    (fp_text reference P2 (at 0 3.81 270) (layer B.SilkS)
+    (fp_text reference P2 (at 0 3.81 270) (layer B.SilkS) hide
       (effects (font (size 1.27 1.27) (thickness 0.2032)) (justify mirror))
     )
@@
     (descr "1 pin")
     (tags "CONN DEV")
-    (fp_text reference P4 (at 0 3.81 270) (layer B.SilkS)
+    (fp_text reference P4 (at 0 3.81 270) (layer B.SilkS) hide
       (effects (font (size 1.27 1.27) (thickness 0.2032)) (justify mirror))
     )
@@
     (descr "1 pin")
     (tags "CONN DEV")
-    (fp_text reference P6 (at 0 3.81 270) (layer B.SilkS)
+    (fp_text reference P6 (at 0 3.81 270) (layer B.SilkS) hide
       (effects (font (size 1.27 1.27) (thickness 0.2032)) (justify mirror))
     )
@@
     (tags "resistor 0805")
     (attr smd)
-    (fp_text reference R2 (at -3 0 360) (layer F.SilkS)
+    (fp_text reference R2 (at -3.1 1.9 360) (layer F.SilkS)
       (effects (font (size 1 1) (thickness 0.15)))
     )
@@
     (tags "resistor 0805")
     (attr smd)
-    (fp_text reference R3 (at 3.5 -1.25 270) (layer F.SilkS)
+    (fp_text reference R3 (at -3.5 0.2 360) (layer F.SilkS)
       (effects (font (size 1 1) (thickness 0.15)))
     )
@@
     (tags "resistor 0805")
     (attr smd)
-    (fp_text reference R4 (at -2.4 2.15 180) (layer F.SilkS)
+    (fp_text reference R4 (at 3.7 -0.2 180) (layer F.SilkS)
       (effects (font (size 1 1) (thickness 0.15)))
     )
@@
     (tags "resistor 0805")
     (attr smd)
-    (fp_text reference R6 (at 0 -2.1 360) (layer F.SilkS)
+    (fp_text reference R6 (at -3.3 1.3 360) (layer F.SilkS)
       (effects (font (size 1 1) (thickness 0.15)))
     )
@@
     )
   )
+  (gr_line (start 150 113) (end 150 116) (angle 90) (layer F.SilkS) (width 0.2))
+  (gr_line (start 157 113) (end 150 113) (angle 90) (layer F.SilkS) (width 0.2))
+  (gr_line (start 157 116) (end 157 113) (angle 90) (layer F.SilkS) (width 0.2))
+  (gr_line (start 150 116) (end 157 116) (angle 90) (layer F.SilkS) (width 0.2))
+  (gr_line (start 124 113) (end 124 116) (angle 90) (layer F.SilkS) (width 0.2))
+  (gr_line (start 131 113) (end 124 113) (angle 90) (layer F.SilkS) (width 0.2))
+  (gr_line (start 131 116) (end 131 113) (angle 90) (layer F.SilkS) (width 0.2))
+  (gr_line (start 124 116) (end 131 116) (angle 90) (layer F.SilkS) (width 0.2))
+  (gr_line (start 97 113) (end 97 116) (angle 90) (layer F.SilkS) (width 0.2))
+  (gr_line (start 104 113) (end 97 113) (angle 90) (layer F.SilkS) (width 0.2))
+  (gr_line (start 104 116) (end 104 113) (angle 90) (layer F.SilkS) (width 0.2))
+  (gr_line (start 97 116) (end 104 116) (angle 90) (layer F.SilkS) (width 0.2))
+  (gr_text 2 (at 96.1 106.8) (layer B.SilkS)
+    (effects (font (size 1.5 1.5) (thickness 0.3)) (justify mirror))
+  )
+  (gr_text 1 (at 96.2 103.9) (layer B.SilkS)
+    (effects (font (size 1.5 1.5) (thickness 0.3)) (justify mirror))
+  )
+  (gr_text 0 (at 96.2 101.7) (layer B.SilkS)
+    (effects (font (size 1.5 1.5) (thickness 0.3)))
+  )
+  (gr_text "BBB -> Pololu" (at 129.9 124) (layer F.SilkS)
+    (effects (font (size 2.5 2.4) (thickness 0.3)))
+  )
   (gr_text Z (at 114.5 120.75) (layer F.SilkS)
